Commit message: Update to use new robot body

File: description/common_dimensions.xacro (robot description, xacro)
@@ -1,14 +1,15 @@
 <?xml version="1.0"?>
 <robot xmlns:xacro="http://www.ros.org/wiki/xacro" >
-    <xacro:property name="chassis_length_x" value="0.55" />
-    <xacro:property name="chassis_width_y" value="0.35" />
-    <xacro:property name="chassis_height_z" value="0.215" />
+    <xacro:property name="in_to_m" value="0.0254" />
+    <xacro:property name="chassis_length_x" value="${20 * in_to_m}" />
+    <xacro:property name="chassis_width_y" value="${12.5 * in_to_m}" />
+    <xacro:property name="chassis_height_z" value="${6.5 * in_to_m}" />
     <xacro:property name="cor_to_rear_of_chassis" value="0.12" />
-    <xacro:property name="front_of_chassis_to_caster" value="0.115" />
+    <xacro:property name="front_of_chassis_to_caster" value="${3 * in_to_m}" />
     <xacro:property name="motor_length" value="0.1" />
     <xacro:property name="wheel_radius" value="0.035" />
     <xacro:property name="wheel_length" value="0.02" />
     <xacro:property name="caster_height" value="${wheel_radius * 2}" />
-    <xacro:property name="inter_motor_distance" value="0.15" />
+    <xacro:property name="inter_motor_distance" value="${4 * in_to_m}" />
     <xacro:property name="robot_height" value="${chassis_height_z + wheel_radius * 2}" />
 </robot>

File: description/lidar.xacro (robot description, xacro)
@@ -4,5 +4,5 @@
         <parent link="chassis" />
         <child link="laser_frame"/>
-        <origin xyz = "${chassis_length_x / 2} 0 ${robot_height + wheel_length / 2 + camera_height}" rpy="0 0 0" />
+        <origin xyz = "${(chassis_length_x / 2)} 0 ${robot_height + wheel_length / 2 + camera_height}" rpy="0 0 0" />
     </joint>
     <link name="laser_frame">
