Commit message: Prevent imu box from clipping into the floor

File: description/imu.xacro (robot description, xacro)
@@ -4,10 +4,10 @@
         <visual>
             <geometry>
-                <box size="0.1 0.1 0.1"/>
+                <box size="0.0001 0.0001 0.0001"/>
             </geometry>
         </visual>
         <collision>
             <geometry>
-                <box size="0.1 0.1 0.1"/>
+                <box size="0.0001 0.0001 0.0001"/>
             </geometry>
         </collision>
@@ -15,5 +15,5 @@
     </link>
     <joint name="imu_joint" type="fixed">
-        <parent link="base_link"/>
+        <parent link="chassis"/>
         <child link="imu_link"/>
         <origin xyz="0 0 0.01"/>
